Commit message: Added other sensors to gazebo sim to get base odom.  That is now used in the sim.

File: roscopter_sim/xacro/platform.urdf.xacro (robot description, xacro)
@@ -47,3 +47,27 @@
     </plugin>
   </gazebo>
+    <!-- ***************** SENSORS ******************* -->
+  <!-- Ground Truth -->
+  <xacro:include filename="$(find rosflight_plugins)/xacro/odometry_sensor.xacro"/>
+  <xacro:odometry_plugin_macro namespace="${namespace}" parent_link="${namespace}/base_link"/>
+  <!-- IMU -->
+  <xacro:include filename="$(find rosflight_plugins)/xacro/imu.xacro"/>
+  <xacro:imu_plugin_macro namespace="${namespace}" parent_link="${namespace}/base_link"/>
+  <!-- Sonar -->
+  <xacro:include filename="$(find rosflight_plugins)/xacro/sonar.xacro"/>
+  <xacro:Sonar_MB1030
+    namespace="${namespace}"
+    parent_link="${namespace}/base_link"
+    sonar_topic="sonar/data">
+    <origin xyz="0 0 0" rpy="0 1.57 0" />
+  </xacro:Sonar_MB1030>
+  <!-- Barometer -->
+  <xacro:include filename="$(find rosflight_plugins)/xacro/barometer.xacro"/>
+  <xacro:barometer_plugin_macro namespace="${namespace}" parent_link="${namespace}/base_link"/>
+  <!-- Magnetometer -->
+  <xacro:include filename="$(find rosflight_plugins)/xacro/magnetometer.xacro"/>
+  <xacro:magnetometer_plugin_macro namespace="${namespace}" parent_link="${namespace}/base_link"/>
+  <!-- GPS -->
+  <xacro:include filename="$(find rosflight_plugins)/xacro/GPS.xacro"/>
+  <xacro:gps_plugin_macro namespace="${namespace}" parent_link="${namespace}/base_link"/>
 </robot>
